File: hardware.kicad_sch (KiCad schematic)
At the start: 22 parts, among them J1 Conn_Load_Cell, J2 Conn_SW_circuit, J3 Conn_SPI, J4 Conn, U1 XIAO-nRF52840-SMD, U2 NAU7802SGI, U3 TCK108AF

Commit message: finished PCB v0.1
Parts:
- removed C7: C, symbol Device:C
- removed J1: Conn_Load_Cell, symbol Connector:Conn_01x04_Pin
- removed J2: Conn_SW_circuit, symbol Connector:Conn_01x02_Pin
- removed J3: Conn_SPI, symbol Connector:Conn_01x20_Socket
- removed J4: Conn, symbol Connector:Conn_01x20_Socket
- removed R5: 10K, symbol Device:R
- removed R6: R, symbol Device:R
- added J1: Terminal_Loadcell, TerminalBlock_TE-Connectivity:TerminalBlock_TE_282834-4_1x04_P2.54mm_Horizontal, symbol Connector:Screw_Terminal_01x04
- added J2: Terminal_Switch, TerminalBlock_TE-Connectivity:TerminalBlock_TE_282834-2_1x02_P2.54mm_Horizontal, symbol Connector:Screw_Terminal_01x02
- added J3: Conn_SPI, Connector_PinSocket_2.54mm:PinSocket_1x20_P2.54mm_Vertical, symbol Connector_Generic:Conn_01x20
- added J4: Conn_I2C, Connector_PinSocket_2.54mm:PinSocket_1x20_P2.54mm_Vertical, symbol Connector_Generic:Conn_01x20
- added TP1: 5V TestPoint, TestPoint:TestPoint_Pad_D1.5mm, symbol Connector:TestPoint
- C1, C2, C3, C4, C5: footprint (none) -> Capacitor_SMD:C_1206_3216Metric_Pad1.33x1.80mm_HandSolder
- C6: value C -> 1uF; footprint (none) -> Capacitor_SMD:C_1206_3216Metric_Pad1.33x1.80mm_HandSolder
- D1: footprint (none) -> LED_SMD:LED_1206_3216Metric_Pad1.42x1.75mm_HandSolder
- R1, R2: value R? -> 47R; footprint (none) -> Resistor_SMD:R_1206_3216Metric_Pad1.30x1.75mm_HandSolder
- R3, R4: footprint (none) -> Resistor_SMD:R_1206_3216Metric_Pad1.30x1.75mm_HandSolder
- R6: renamed from R7; value R? -> 50R; footprint (none) -> Resistor_SMD:R_1206_3216Metric_Pad1.30x1.75mm_HandSolder
- U1: footprint MCU_SEEED_XIAO_Series:XIAO-nRF52840-SMD -> Seeed Studio XIAO Series Library:XIAO-nRF52840-SMD
- U2: footprint SOI16_NAU7802SGI_NUV -> Library:SOI16_NAU7802SGI_NUV
Connections:
- net +3V3: now also C6.1, J3.2 (Pin_2); no longer C1.1, C2.1, U2.1 (REFP)
- net A+: now also J1.4 (Pin_4)
- net A-: now also J1.3 (Pin_3)
- net GND: now also C6.2, U1.16 (GND), U1.22 (GND), J1.2 (Pin_2), J3.1 (Pin_1), J3.11 (Pin_11), J4.20 (Pin_20), J4.9 (Pin_9)
- net +5V: no longer names the net of U1.14 (5V)
- net +5V: now also TP1.1
- net AVDD renamed Exc_Pos
- net Exc_Pos: now also C1.1, C2.1, U2.1 (REFP), J1.1 (Pin_1)
- net CNT renamed PA2_CNT
- net CS renamed PB9_CS
- net PB9_CS: now also J3.7 (Pin_7)
- net DRDY renamed PA10_SDA
- net PA10_SDA: now also R3.2, U2.14 (SDIO), J4.10 (Pin_10); no longer U2.12 (DRDY)
- net D/C renamed PB8_D/C
- net PB8_D/C: now also J3.8 (Pin_8)
- net IRQ renamed PA11_SCL
- net PA11_SCL: now also R4.2, U2.13 (SCLK), J4.11 (Pin_11)
- net MISO renamed PA5_MISO
- net PA5_MISO: now also J3.5 (Pin_5)
- net MOSI renamed PA6_SCK
- net PA6_SCK: now also J3.4 (Pin_4)
- net PA4_LED renamed PA2_LED
- net PA2_LED: now also U1.6 (PA9_A5_D5_SCL); no longer U1.2 (PA4_A1_D1)
- net PWR+ renamed SW_In
- net SW_In: now also J2.1 (Pin_1)
- net PWR- renamed SW_Out
- net SW_Out: now also J2.2 (Pin_2)
- net SCK renamed PA7_MOSI
- net PA7_MOSI: now also J3.6 (Pin_6)
- removed net SCL: R4.2, U1.6 (PA9_A5_D5_SCL), U2.13 (SCLK)
- removed net SDA: R3.2, U1.5 (PA8_A4_D4_SDA), U2.14 (SDIO)
- new net PA4_IRQ: J4.12 (Pin_12), U1.2 (PA4_A1_D1)
- new net PA8_DRDY: U1.5 (PA8_A4_D4_SDA), U2.12 (DRDY)
- no-connect marks 27 -> 35
Other:
- title: Rocket Gravimetric Espresso -> Rocket Gravimetric Espresso Schematic
- moved on the sheet: C1, C2, C3, C4, C5, R1, R2, R3, R4, U1
